File: Business Card.kicad_pcb (KiCad board)
At the start: 2 copper layers, 88.9 x 50.8 mm, 71 parts, among them Q1 AO3401A, U1 ATtiny1616-M, U2 NT3H2111W0FHKH

Commit message: Board Edited
Routing:
- net Net-(U2-VCC): track 4.95 -> 6.64 mm
Changed lines of the file:
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@@
     (property "SnapEDA_Link" "https://www.snapeda.com/parts/NT3H2111W0FHKH/NXP+USA+Inc./view-part/?ref=snap")
     (attr smd)
-    (fp_text reference "U2" (at 2.4812 -0.0092) (layer "F.SilkS")
+    (fp_text reference "U2" (at 2.786 -0.441) (layer "F.SilkS")
         (effects (font (size 0.800953 0.800953) (thickness 0.15)))
     )
@@
   (gr_line (start 156.718 88.9) (end 156.718 95.504)
     (stroke (width 0.1) (type default)) (layer "Edge.Cuts"))
-  (gr_rect (start 96.52 121.92) (end 185.42 71.12)
+  (gr_rect (start 96.52 71.12) (end 185.42 121.92)
     (stroke (width 0.1) (type default)) (fill none) (layer "Edge.Cuts"))
   (gr_line (start 159.258 86.36) (end 156.718 88.9)
@@
   (segment (start 169.87 115.824) (end 165.41 115.824) (width 0.25) (layer "F.Cu") (net 7))
   (segment (start 171.704 113.99) (end 169.87 115.824) (width 0.25) (layer "F.Cu") (net 7))
-  (segment (start 125.073 110.354) (end 125.717 110.998) (width 0.25) (layer "F.Cu") (net 11))
-  (segment (start 125.668 107.375) (end 125.386 107.375) (width 0.25) (layer "F.Cu") (net 11))
-  (segment (start 125.386 107.375) (end 125.073 107.687) (width 0.25) (layer "F.Cu") (net 11))
-  (segment (start 125.073 107.687) (end 125.073 110.354) (width 0.25) (layer "F.Cu") (net 11))
+  (segment (start 124.968 110.249) (end 125.717 110.998) (width 0.25) (layer "F.Cu") (net 11))
+  (segment (start 125.194422 107.385) (end 124.955 107.624422) (width 0.25) (layer "F.Cu") (net 11))
+  (segment (start 125.72 107.385) (end 125.194422 107.385) (width 0.25) (layer "F.Cu") (net 11))
+  (segment (start 124.955 107.624422) (end 124.955 108.145578) (width 0.25) (layer "F.Cu") (net 11))
+  (segment (start 124.955 108.145578) (end 124.968 108.158578) (width 0.25) (layer "F.Cu") (net 11))
+  (segment (start 124.968 108.158578) (end 124.968 110.249) (width 0.25) (layer "F.Cu") (net 11))
   (segment (start 125.805 107.375) (end 125.798 107.375) (width 0.25) (layer "F.Cu") (net 11))
-  (segment (start 125.668 107.375) (end 125.798 107.375) (width 0.2198) (layer "F.Cu") (net 11))
-  (segment (start 127.195 106.875) (end 127.195 107.375) (width 0.25) (layer "F.Cu") (net 12))
-  (segment (start 127.904 110.361) (end 127.267 110.998) (width 0.25) (layer "F.Cu") (net 12))
-  (segment (start 127.195 107.375) (end 127.656 107.375) (width 0.25) (layer "F.Cu") (net 12))
-  (segment (start 127.656 107.375) (end 127.904 107.623) (width 0.25) (layer "F.Cu") (net 12))
-  (segment (start 127.904 107.623) (end 127.904 110.361) (width 0.25) (layer "F.Cu") (net 12))
+  (segment (start 127.949 107.375) (end 128.27 107.696) (width 0.25) (layer "F.Cu") (net 12))
+  (segment (start 127.949 107.375) (end 127.195 107.375) (width 0.25) (layer "F.Cu") (net 12))
+  (segment (start 128.27 107.696) (end 128.27 107.188) (width 0.25) (layer "F.Cu") (net 12))
+  (segment (start 127.267 110.998) (end 128.27 109.995) (width 0.25) (layer "F.Cu") (net 12))
+  (segment (start 128.27 107.188) (end 127.957 106.875) (width 0.25) (layer "F.Cu") (net 12))
+  (segment (start 127.957 106.875) (end 127.195 106.875) (width 0.25) (layer "F.Cu") (net 12))
+  (segment (start 128.27 109.995) (end 128.27 107.696) (width 0.25) (layer "F.Cu") (net 12))
   (segment (start 126.5 104.386) (end 126.5 103.386) (width 0.25) (layer "F.Cu") (net 13))
   (segment (start 124.968 101.854) (end 124.968 96.774) (width 0.25) (layer "F.Cu") (net 13))
@@
   (segment (start 126.5 104.402) (end 126.492 104.394) (width 0.25) (layer "F.Cu") (net 13))
   (segment (start 126.5 106.68) (end 126.5 104.402) (width 0.25) (layer "F.Cu") (net 13))
-  (segment (start 125.805 106.875) (end 124.968 106.038) (width 0.25) (layer "F.Cu") (net 14))
-  (segment (start 124.968 106.038) (end 124.968 104.394) (width 0.25) (layer "F.Cu") (net 14))
+  (segment (start 125.805 106.875) (end 125.163 106.875) (width 0.25) (layer "F.Cu") (net 14))
+  (segment (start 124.968 106.68) (end 124.968 104.394) (width 0.25) (layer "F.Cu") (net 14))
+  (segment (start 125.163 106.875) (end 124.968 106.68) (width 0.25) (layer "F.Cu") (net 14))
   (via (at 124.968 104.394) (size 0.8) (drill 0.4) (layers "F.Cu" "B.Cu") (net 14))
   (segment (start 119.38 98.806) (end 119.38 97.155) (width 0.25) (layer "B.Cu") (net 14))
@@
   (segment (start 138.156 84.074) (end 138.156 83.586) (width 0.2) (layer "F.Cu") (net 16))
   (segment (start 132.842 82.296) (end 130.302 82.296) (width 0.2) (layer "F.Cu") (net 16))
-  (segment (start 156.3518 99.2992) (end 156.352 99.2992) (width 0.2) (layer "F.Cu") (net 17))
   (segment (start 169.87 108.43) (end 165.41 108.43) (width 0.2) (layer "F.Cu") (net 17))
-  (segment (start 156.604 99.0469) (end 156.352 99.2992) (width 0.2) (layer "F.Cu") (net 17))
   (segment (start 165.41 108.43) (end 164.007 108.43) (width 0.2) (layer "F.Cu") (net 17))
-  (segment (start 157.764 99.0469) (end 156.604 99.0469) (width 0.2) (layer "F.Cu") (net 17))
+  (segment (start 157.764 99.0469) (end 157.5117 99.2992) (width 0.2) (layer "F.Cu") (net 17))
+  (segment (start 157.5117 99.2992) (end 156.3518 99.2992) (width 0.2) (layer "F.Cu") (net 17))
   (via (at 157.764 99.0469) (size 0.8) (drill 0.4) (layers "F.Cu" "B.Cu") (net 17))
   (via (at 164.007 108.43) (size 0.8) (drill 0.4) (layers "F.Cu" "B.Cu") (net 17))
@@
   (segment (start 177.606 101.811) (end 177.606 113.31) (width 0.2) (layer "F.Cu") (net 18))
   (segment (start 173.99 100.584) (end 174.075 100.499) (width 0.2) (layer "F.Cu") (net 18))
-  (segment (start 156.352 101.4252) (end 156.352 111.988) (width 0.2) (layer "F.Cu") (net 19))
+  (segment (start 157.48 101.092) (end 157.2872 100.8992) (width 0.2) (layer "F.Cu") (net 19))
   (segment (start 162.814 113.99) (end 158.354 113.99) (width 0.2) (layer "F.Cu") (net 19))
-  (segment (start 156.352 111.988) (end 158.354 113.99) (width 0.2) (layer "F.Cu") (net 19))
-  (segment (start 156.352 100.899) (end 156.352 101.4252) (width 0.2) (layer "F.Cu") (net 19))
-  (segment (start 156.352 101.4252) (end 156.3518 101.425) (width 0.2) (layer "F.Cu") (net 19))
-  (segment (start 156.3518 101.425) (end 156.3518 100.8992) (width 0.2) (layer "F.Cu") (net 19))
+  (segment (start 158.354 113.99) (end 157.226 112.862) (width 0.2) (layer "F.Cu") (net 19))
+  (segment (start 157.226 112.862) (end 157.226 102.2992) (width 0.2) (layer "F.Cu") (net 19))
+  (segment (start 157.48 102.0452) (end 157.48 101.092) (width 0.2) (layer "F.Cu") (net 19))
+  (segment (start 157.226 102.2992) (end 157.48 102.0452) (width 0.2) (layer "F.Cu") (net 19))
+  (segment (start 157.2872 100.8992) (end 156.3518 100.8992) (width 0.2) (layer "F.Cu") (net 19))
   (segment (start 169.87 119.324) (end 165.41 119.324) (width 0.2) (layer "F.Cu") (net 20))
   (segment (start 155.7018 102.1078) (end 155.7018 101.5492) (width 0.2) (layer "F.Cu") (net 20))
